File: Board/GCtoUSB_Current.sch (EAGLE design)
At the start: 40 parts, among them J1 AVR_SPI_PRG_6PTH, J2 AVR_SPI_PRG_6PTH, U1 ATMEGA8U2AU, U2 3.3V_REG_LDOSMD, X1 USB-MB-H, Y1 16MHz, Y2 16MHz

Commit message: Moved to eagle 6.2. Completed SMT version of board - now saved as version 1.3.
Parts:
- U1: value ATMEGA8U2AU -> 8U2
- ZIC1: value ATMEGA328 -> 328
